Commit message: update

File: config/fisheye_stereo.urdf.xacro (robot description, xacro)
@@ -1,10 +1,9 @@
 <?xml version="1.0"?>
-<robot name="sensor_fisheye" xmlns:xacro="http://ros.org/wiki/xacro">
+<robot name="sensor_stereo" xmlns:xacro="http://ros.org/wiki/xacro">
   <xacro:include filename="$(find turtlebot_description)/urdf/turtlebot_gazebo_fisheye_stereo.urdf.xacro"/>
-  <!-- <xacro:include filename="$(find turtlebot_description)/urdf/turtlebot_properties.urdf.xacro"/> -->
   <xacro:include filename="$(find turtlebot_description)/urdf/turtlebot_properties_fisheye_stereo.urdf.xacro"/>
   <xacro:property name="fisheye_cam_py" value="-0.05"/>
   <!-- Parameterised in part by the values in turtlebot_properties.urdf.xacro -->
-  <xacro:macro name="sensor_fisheye" params="parent">
+  <xacro:macro name="sensor_stereo" params="parent">
     <joint name="camera_left_joint" type="fixed">
       <origin xyz="${cam_px} ${fisheye_cam_py} ${cam_pz}" rpy="${cam_or} ${cam_op} ${cam_oy}"/>
@@ -19,14 +18,14 @@
     </joint>
     <link name="camera_left_optical_frame"/>
-    <joint name="camera_joint" type="fixed">
-      <origin xyz="0 -${fisheye_cam_py} 0" rpy="0 0 0"/>
+    <joint name="camera_joint_1" type="fixed">
+      <origin xyz="0 ${-fisheye_cam_py} 0" rpy="0 0 0"/>
       <parent link="camera_left_frame"/>
-      <child link="camera_link"/>
+      <child link="camera_link_1"/>
     </joint>
-      <link name="camera_link">
+      <link name="camera_link_1">
       <visual>
        <origin xyz="0 0 0" rpy="0 0 ${M_PI/2}"/>
         <geometry>
-         <mesh filename="package://turtlebot_description/meshes/sensors/r200.dae"/>
+         <mesh filename="package://turtlebot_description/meshes/sensors/kinect.dae"/>
         </geometry>
       </visual>
@@ -49,5 +48,5 @@
          (Hence, don't publish them additionally!) -->
   <joint name="camera_right_joint" type="fixed">
-    <origin xyz="0 -2*${fisheye_cam_py} 0" rpy="0 0 0" />
+    <origin xyz="0 ${2 * -fisheye_cam_py} 0" rpy="0 0 0" />
     <parent link="camera_left_frame" />
     <child link="camera_right_frame" />
@@ -61,5 +60,5 @@
   <link name="camera_right_optical_joint"/>
   <!-- Kinect sensor for simulation -->
-  <turtlebot_sim_3dsensor/>
+  <turtlebot_sim_stereo_sensor/>
   </xacro:macro>
 </robot>

File: config/kobuki_hexagons_fisheye_stereo_ADIS_16448.urdf.xacro (robot description, xacro)
@@ -10,9 +10,9 @@
   <xacro:include filename="$(find kobuki_description)/urdf/kobuki_ADIS_16448.urdf.xacro" />
   <xacro:include filename="$(find turtlebot_description)/urdf/stacks/hexagons.urdf.xacro"/>
-  <xacro:include filename="$(find turtlebot_description)/urdf/sensors/kinect.urdf.xacro"/>
+  <!-- <xacro:include filename="$(find turtlebot_description)/urdf/sensors/kinect.urdf.xacro"/>  -->
   <xacro:include filename="$(find turtlebot_description)/urdf/sensors/fisheye_stereo.urdf.xacro"/>
   <kobuki/>
   <stack_hexagons parent="base_link"/>
-  <sensor_kinect  parent="base_link"/>
-  <sensor_camera  parent="base_link"/>
+  <!-- <sensor_kinect  parent="base_link"/> -->
+  <sensor_stereo  parent="base_link"/>
 </robot>

File: config/kobuki_hexagons_fisheye_stereo_mpu_6000.urdf.xacro (robot description, xacro)
@@ -10,9 +10,9 @@
   <xacro:include filename="$(find kobuki_description)/urdf/kobuki_mpu_6000.urdf.xacro" />
   <xacro:include filename="$(find turtlebot_description)/urdf/stacks/hexagons.urdf.xacro"/>
-  <xacro:include filename="$(find turtlebot_description)/urdf/sensors/kinect.urdf.xacro"/>
+  <!-- <xacro:include filename="$(find turtlebot_description)/urdf/sensors/kinect.urdf.xacro"/>  -->
   <xacro:include filename="$(find turtlebot_description)/urdf/sensors/fisheye_stereo.urdf.xacro"/>
   <kobuki/>
   <stack_hexagons parent="base_link"/>
-  <sensor_kinect  parent="base_link"/>
-  <sensor_camera  parent="base_link"/>
+  <!-- <sensor_kinect  parent="base_link"/> -->
+  <sensor_stereo  parent="base_link"/>
 </robot>

File: config/turtlebot_gazebo_fisheye_stereo.urdf.xacro (robot description, xacro)
@@ -2,6 +2,6 @@
 <robot name="turtlebot_gazebo" xmlns:xacro="http://ros.org/wiki/xacro">
   <!-- Microsoft Kinect / ASUS Xtion PRO Live for simulation -->
-  <xacro:macro name="turtlebot_sim_3dsensor">
-    <gazebo reference="camera_link">
+  <xacro:macro name="turtlebot_sim_stereo_sensor">
+    <gazebo reference="camera_link_1">
     <sensor type="multicamera" name="stereo_camera">
       <always_on>true</always_on>

Commit message: freeze

File: config/fisheye_stereo.urdf.xacro (robot description, xacro)
@@ -3,5 +3,6 @@
   <xacro:include filename="$(find turtlebot_description)/urdf/turtlebot_gazebo_fisheye_stereo.urdf.xacro"/>
   <xacro:include filename="$(find turtlebot_description)/urdf/turtlebot_properties_fisheye_stereo.urdf.xacro"/>
-  <xacro:property name="fisheye_cam_py" value="-0.05"/>
+  <!-- <xacro:property name="fisheye_cam_py" value="-0.05"/> -->
+  <xacro:property name="fisheye_cam_py" value="-0.0125"/>
   <!-- Parameterised in part by the values in turtlebot_properties.urdf.xacro -->
   <xacro:macro name="sensor_stereo" params="parent">
@@ -19,5 +20,6 @@
     <link name="camera_left_optical_frame"/>
     <joint name="camera_joint_1" type="fixed">
-      <origin xyz="0 ${-fisheye_cam_py} 0" rpy="0 0 0"/>
+      <!-- <origin xyz="0 ${-fisheye_cam_py} 0" rpy="0 0 0"/> -->
+      <origin xyz="-0.031 ${-fisheye_cam_py} -0.016" rpy="0 0 0"/>
       <parent link="camera_left_frame"/>
       <child link="camera_link_1"/>

File: config/turtlebot_gazebo_fisheye_stereo.urdf.xacro (robot description, xacro)
@@ -15,5 +15,5 @@
         </image>
         <clip>
-          <near>0.02</near>
+          <near>0.05</near>
           <far>50</far>
         </clip>
@@ -33,5 +33,5 @@
         </image>
         <clip>
-          <near>0.02</near>
+          <near>0.05</near>
           <far>50</far>
         </clip>
@@ -43,8 +43,8 @@
       </camera>
       <plugin name="stereo_camera_controller" filename="libgazebo_ros_multicamera.so">
+        <cameraName>multisense_sl/camera</cameraName>
         <alwaysOn>true</alwaysOn>
         <!-- ATTENTION keep the update rate as it is for customed fps!!! -->
         <updateRate>0.0</updateRate>
-        <cameraName>multisense_sl/camera</cameraName>
         <imageTopicName>image_raw</imageTopicName>
         <cameraInfoTopicName>camera_info</cameraInfoTopicName>

File: config/turtlebot_properties.urdf.xacro (robot description, xacro)
@@ -19,9 +19,9 @@
      (currently in development and awaiting feedback)
    -->
-	<xacro:property name="cam_px" value="0.15" />
-	<xacro:property name="cam_pz" value="0.3" />
-	<xacro:property name="cam_or" value="0" />
-	<xacro:property name="cam_op" value="0" />
-	<xacro:property name="cam_oy" value="0" />
+  <xacro:property name="cam_px" value="0.15" />
+  <xacro:property name="cam_pz" value="0.3" />
+  <xacro:property name="cam_or" value="0" />
+  <xacro:property name="cam_op" value="0" />
+  <xacro:property name="cam_oy" value="0" />
 <!--   <xacro:property name="cam_px" value="-0.087" />
   <xacro:property name="cam_pz" value="0.2870" />

Commit message: update

File: config/fisheye_stereo.urdf.xacro (robot description, xacro)
@@ -50,5 +50,5 @@
          (Hence, don't publish them additionally!) -->
   <joint name="camera_right_joint" type="fixed">
-    <origin xyz="0 ${2 * -fisheye_cam_py} 0" rpy="0 0 0" />
+    <origin xyz="0 -0.11 0" rpy="0 0 0" />
     <parent link="camera_left_frame" />
     <child link="camera_right_frame" />
@@ -58,7 +58,7 @@
     <origin xyz="0 0 0" rpy="${-M_PI/2} 0 ${-M_PI/2}" />
     <parent link="camera_right_frame" />
-    <child link="camera_right_optical_joint" />
+    <child link="camera_right_optical_frame" />
   </joint>
-  <link name="camera_right_optical_joint"/>
+  <link name="camera_right_optical_frame"/>
   <!-- Kinect sensor for simulation -->
   <turtlebot_sim_stereo_sensor/>

Commit message: use pinhole stereo instead

File: config/fisheye_stereo.urdf.xacro (robot description, xacro)
@@ -3,5 +3,4 @@
   <xacro:include filename="$(find turtlebot_description)/urdf/turtlebot_gazebo_fisheye_stereo.urdf.xacro"/>
   <xacro:include filename="$(find turtlebot_description)/urdf/turtlebot_properties_fisheye_stereo.urdf.xacro"/>
-  <!-- <xacro:property name="fisheye_cam_py" value="-0.05"/> -->
   <xacro:property name="fisheye_cam_py" value="-0.0125"/>
   <!-- Parameterised in part by the values in turtlebot_properties.urdf.xacro -->
@@ -29,5 +28,5 @@
        <origin xyz="0 0 0" rpy="0 0 ${M_PI/2}"/>
         <geometry>
-         <mesh filename="package://turtlebot_description/meshes/sensors/kinect.dae"/>
+         <mesh filename="package://turtlebot_description/meshes/sensors/r200.dae"/>
         </geometry>
       </visual>
@@ -50,5 +49,6 @@
          (Hence, don't publish them additionally!) -->
   <joint name="camera_right_joint" type="fixed">
-    <origin xyz="0 -0.11 0" rpy="0 0 0" />
+    <origin xyz="0 ${-stereo_baseline} 0" rpy="0 0 0" />
+	  <!-- <origin xyz="0 ${2 * -fisheye_cam_py} 0" rpy="0 0 0" /> -->
     <parent link="camera_left_frame" />
     <child link="camera_right_frame" />

File: config/turtlebot_gazebo_fisheye_stereo.urdf.xacro (robot description, xacro)
@@ -2,4 +2,5 @@
 <robot name="turtlebot_gazebo" xmlns:xacro="http://ros.org/wiki/xacro">
   <!-- Microsoft Kinect / ASUS Xtion PRO Live for simulation -->
+  <xacro:property name="stereo_baseline" value="0.11"/>
   <xacro:macro name="turtlebot_sim_stereo_sensor">
     <gazebo reference="camera_link_1">
@@ -25,5 +26,5 @@
       </camera>
       <camera name="right">
-        <pose>0 -0.11 0 0 0 0</pose>
+        <pose>0 ${-stereo_baseline} 0 0 0 0</pose>
         <horizontal_fov>1.61408657</horizontal_fov>
         <image>
@@ -51,21 +52,21 @@
         <frameName>left_camera_optical_frame</frameName>
         <!--<rightFrameName>right_camera_optical_frame</rightFrameName>-->
-        <hackBaseline>0.11</hackBaseline>
-        <CxPrime>406.6650580307593</CxPrime>
-        <Cx>406.6650580307593</Cx>
-        <Cy>256.20533579714373</Cy>
+        <hackBaseline>${stereo_baseline}</hackBaseline>
+        <CxPrime>376</CxPrime>
+        <Cx>376</Cx>
+        <Cy>240</Cy>
         <!-- image_width / (2*tan(hfov_radian /2)) 360.0652897865692 -->
         <!-- 320 for wide and 772.55 for narrow stereo camera -->
-        <focal_length>360.0652897865692</focal_length>
-        <distortionK1>-0.27186431380704884</distortionK1>
+        <focal_length>360.06528871</focal_length>
+        <!-- <distortionK1>-0.27186431380704884</distortionK1>
         <distortionK2>0.05397709169334604</distortionK2>
         <distortionK3>-0.000557307377524114</distortionK3>
         <distortionT1>-0.0006127379205397152</distortionT1>
-        <distortionT2>0.0</distortionT2>
-<!--         <distortionK1>0.0</distortionK1>
+        <distortionT2>0.0</distortionT2> -->
+        <distortionK1>0.0</distortionK1>
         <distortionK2>0.0</distortionK2>
         <distortionK3>0.0</distortionK3>
         <distortionT1>0.0</distortionT1>
-        <distortionT2>0.0</distortionT2> -->
+        <distortionT2>0.0</distortionT2>
       </plugin>
     </sensor>

Commit message: update

File: config/fisheye_stereo.urdf.xacro (robot description, xacro)
@@ -6,20 +6,20 @@
   <!-- Parameterised in part by the values in turtlebot_properties.urdf.xacro -->
   <xacro:macro name="sensor_stereo" params="parent">
-    <joint name="camera_left_joint" type="fixed">
+    <joint name="left_camera_joint" type="fixed">
       <origin xyz="${cam_px} ${fisheye_cam_py} ${cam_pz}" rpy="${cam_or} ${cam_op} ${cam_oy}"/>
       <parent link="${parent}"/>
-      <child link="camera_left_frame" />
+      <child link="left_camera_frame" />
     </joint>
-    <link name="camera_left_frame"/>
-    <joint name="camera_left_optical_joint" type="fixed">
+    <link name="left_camera_frame"/>
+    <joint name="left_camera_optical_joint" type="fixed">
       <origin xyz="0 0 0" rpy="${-M_PI/2} 0 ${-M_PI/2}" />
-      <parent link="camera_left_frame" />
-      <child link="camera_left_optical_frame" />
+      <parent link="left_camera_frame" />
+      <child link="left_camera_optical_frame" />
     </joint>
-    <link name="camera_left_optical_frame"/>
+    <link name="left_camera_optical_frame"/>
     <joint name="camera_joint_1" type="fixed">
       <!-- <origin xyz="0 ${-fisheye_cam_py} 0" rpy="0 0 0"/> -->
       <origin xyz="-0.031 ${-fisheye_cam_py} -0.016" rpy="0 0 0"/>
-      <parent link="camera_left_frame"/>
+      <parent link="left_camera_frame"/>
       <child link="camera_link_1"/>
     </joint>
@@ -48,17 +48,17 @@
          files. However, for Gazebo simulation we need them, so we add them here.
          (Hence, don't publish them additionally!) -->
-  <joint name="camera_right_joint" type="fixed">
+  <joint name="right_camera_joint" type="fixed">
     <origin xyz="0 ${-stereo_baseline} 0" rpy="0 0 0" />
-	  <!-- <origin xyz="0 ${2 * -fisheye_cam_py} 0" rpy="0 0 0" /> -->
-    <parent link="camera_left_frame" />
-    <child link="camera_right_frame" />
+    <!-- <origin xyz="0 ${2 * -fisheye_cam_py} 0" rpy="0 0 0" /> -->
+    <parent link="left_camera_frame" />
+    <child link="right_camera_frame" />
   </joint>
-  <link name="camera_right_frame"/>
-  <joint name="camera_right_optical_joint" type="fixed">
+  <link name="right_camera_frame"/>
+  <joint name="right_camera_optical_joint" type="fixed">
     <origin xyz="0 0 0" rpy="${-M_PI/2} 0 ${-M_PI/2}" />
-    <parent link="camera_right_frame" />
-    <child link="camera_right_optical_frame" />
+    <parent link="right_camera_frame" />
+    <child link="right_camera_optical_frame" />
   </joint>
-  <link name="camera_right_optical_frame"/>
+  <link name="right_camera_optical_frame"/>
   <!-- Kinect sensor for simulation -->
   <turtlebot_sim_stereo_sensor/>
