Commit message: Arrange scripts and launch files

File: config/urdf/kobuki_hexagons_fisheye_stereo_mpu_6000_laser.urdf.xacro (robot description, xacro)
@@ -11,8 +11,8 @@
   <xacro:include filename="$(find turtlebot_description)/urdf/stacks/hexagons.urdf.xacro"/>
   <xacro:include filename="$(find turtlebot_description)/urdf/sensors/fisheye_stereo.urdf.xacro"/>
-  <xacro:include filename="$(find turtlebot_description)/urdf/sensors/hokuyo.urdf.xacro"/>
+  <xacro:include filename="$(find turtlebot_description)/urdf/sensors/laser.urdf.xacro"/>
   <xacro:kobuki/>
   <xacro:stack_hexagons parent="base_link"/>
   <xacro:sensor_stereo  parent="base_link"/>
-  <xacro:sensor_hokuyo  parent="base_link"/>
+  <xacro:sensor_laser   parent="base_link"/>
 </robot>

File: config/urdf/laser.urdf.xacro (robot description, xacro)
@@ -1,17 +1,16 @@
 <?xml version="1.0"?>
-<robot name="sensor_hokuyo" xmlns:xacro="http://ros.org/wiki/xacro">
-  <xacro:include filename="$(find turtlebot_description)/urdf/turtlebot_gazebo_hokuyo.urdf.xacro"/>
-  <xacro:include filename="$(find turtlebot_description)/urdf/turtlebot_properties_hokuyo.urdf.xacro"/>
-  <xacro:property name="hokuyo_py" value="-0.0125"/>
+<robot name="sensor_laser" xmlns:xacro="http://ros.org/wiki/xacro">
+  <xacro:include filename="$(find turtlebot_description)/urdf/turtlebot_gazebo_laser.urdf.xacro"/>
+  <xacro:include filename="$(find turtlebot_description)/urdf/turtlebot_properties_laser.urdf.xacro"/>
   <!-- Parameterised in part by the values in turtlebot_properties.urdf.xacro -->
-  <xacro:macro name="sensor_hokuyo" params="parent">
-    <joint name="hokuyo_joint" type="fixed">
+  <xacro:macro name="sensor_laser" params="parent">
+    <joint name="laser_joint" type="fixed">
       <axis xyz="0 1 0" />
-      <origin xyz="${lidar_px} ${lidar_py} ${lidar_pz}" rpy="${lidar_or} ${lidar_op} ${lidar_oy}"/>
+      <origin xyz="${laser_px} ${laser_py} ${laser_pz}" rpy="${laser_or} ${laser_op} ${laser_oy}"/>
       <parent link="${parent}"/>
-      <child link="hokuyo_link"/>
+      <child link="laser_link"/>
     </joint>
-    <!-- Hokuyo Laser -->
-    <link name="hokuyo_link">
+    <!-- 2D Laser -->
+    <link name="laser_link">
       <collision>
         <origin xyz="0 0 0" rpy="0 0 0"/>
@@ -32,5 +31,5 @@
       </inertial>
     </link>
-    <xacro:turtlebot_sim_hokuyo_sensor/>
+    <xacro:turtlebot_sim_laser_sensor/>
   </xacro:macro>
 </robot>

File: config/urdf/turtlebot_gazebo_laser.urdf.xacro (robot description, xacro)
@@ -1,8 +1,8 @@
 <?xml version="1.0"?>
 <robot name="turtlebot_gazebo" xmlns:xacro="http://ros.org/wiki/xacro">
-  <xacro:macro name="turtlebot_sim_hokuyo_sensor">
-    <!-- hokuyo -->
-    <gazebo reference="hokuyo_link">
-      <sensor type="ray" name="head_hokuyo_sensor">
+  <xacro:macro name="turtlebot_sim_laser_sensor">
+    <!-- laser -->
+    <gazebo reference="laser_link">
+      <sensor type="ray" name="head_laser_sensor">
         <always_on>true</always_on>
         <pose>0 0 0 0 0 0</pose>
@@ -12,18 +12,18 @@
           <scan>
             <horizontal>
-              <samples>666</samples>
+              <samples>3000</samples>
               <resolution>1</resolution>
-              <min_angle>-2.09</min_angle>
-              <max_angle>2.09</max_angle>
+              <min_angle>-3.14</min_angle> # 360 degrees
+              <max_angle>3.14</max_angle>
             </horizontal>
           </scan>
           <range>
             <min>0.10</min>
-            <max>5.6</max>
+            <max>30.0</max>
             <resolution>0.01</resolution>
           </range>
           <noise>
             <type>gaussian</type>
-            <!-- Noise parameters based on published spec for Hokuyo laser
+            <!-- Noise parameters based on published spec for laser
                  achieving "+-30mm" accuracy at range < 10m.  A mean of 0.0m and
                  stddev of 0.01m will put 99.7% of samples within 0.03m of the true
@@ -33,7 +33,7 @@
           </noise>
         </ray>
-        <plugin name="gazebo_ros_head_hokuyo_controller" filename="libgazebo_ros_laser.so">
+        <plugin name="gazebo_ros_head_laser_controller" filename="libgazebo_ros_laser.so">
           <topicName>/scan</topicName>
-          <frameName>hokuyo_link</frameName>
+          <frameName>laser_link</frameName>
         </plugin>
       </sensor>

File: config/urdf/turtlebot_properties_laser.urdf.xacro (robot description, xacro)
@@ -7,9 +7,9 @@
     http://www.ros.org/reps/rep-0119.html
    -->
-	<xacro:property name="lidar_px" value="0.0" />
-	<xacro:property name="lidar_py" value="0.0" />
-	<xacro:property name="lidar_pz" value="0.5" />
-	<xacro:property name="lidar_or" value="0" />
-	<xacro:property name="lidar_op" value="0" />
-	<xacro:property name="lidar_oy" value="0" />
+	<xacro:property name="laser_px" value="0.0" />
+	<xacro:property name="laser_py" value="0.0" />
+	<xacro:property name="laser_pz" value="0.5" />
+	<xacro:property name="laser_or" value="0" />
+	<xacro:property name="laser_op" value="0" />
+	<xacro:property name="laser_oy" value="0" />
 </robot>
